File: board/wmk.kicad_pcb (KiCad board)
At the start: 4 copper layers, 34.5 x 100 mm, 26 parts, among them IC1 LM1117MPX-3.3, J1 Conn_01x03, U2 STM32F103C8T6, X1 PN87520-S

Commit message: gerbers
Parts:
- removed C10, C11: 22p, wmk:C0603
- removed PROGRAMER0: ~, wmk:JP3Q
- removed Q1: ~, wmk:HC49_S
- removed U$1: , wmk:3,3
- added J2: Conn_01x02, Connector_PinHeader_2.54mm:PinHeader_1x02_P2.54mm_Vertical, F.Cu at (157.2, 80.6)
- U2: footprint wmk:QFP50P900X900X160-48N -> Package_QFP:LQFP-48_7x7mm_P0.5mm
- moved JP3 9.36 mm to (151.4, 94.8)
- moved C7 6.74 mm to (149.8, 82.2)
- moved R2 6.65 mm to (149.9, 79.2)
- moved J1 2.69 mm to (158.5, 91.2)
- moved F1 0.56 mm to (158.4, 63.3)
- moved R1 0.40 mm to (154.9, 87.5)
Connections:
- U2 pad 5: Net-(U2-PD0_OSC_IN) -> unconnected-(U2-PD0_OSC_IN-Pad5)
- U2 pad 6: Net-(U2-PD1_OSC_OUT) -> unconnected-(U2-PD1_OSC_OUT-Pad6)
Routing:
- net Net-(U2-PD0_OSC_IN): track 20.9 -> 0.00 mm
- net Net-(U2-PD1_OSC_OUT): track 18.5 -> 0.00 mm
- net /SWCLK: track 33.6 -> 19.5 mm, vias 1 -> 2
- net /RX: track 36.8 -> 28.1 mm
- net /TX: track 42.3 -> 33.8 mm
- net /NRST: track 11.7 -> 5.01 mm, vias 0 -> 1
- net GND: track 27.4 -> 20.9 mm, vias 11 -> 9
- net VDD: track 54.4 -> 49.0 mm
- net /DATA: track 56.9 -> 52.9 mm
- net Net-(J1-Pin_2): track 6.49 -> 3.20 mm, vias 1 -> 0
- net /SWDIO: track 18.1 -> 15.7 mm
- net unconnected-(U2-PA2-Pad12): track 2.01 -> 0.00 mm, vias 1 -> 0
- net /CLOCK: track 44.8 -> 43.3 mm
Other:
- board size 34.5 x 100 mm -> 33.3 x 100 mm

Commit message: initial version
Parts:
- removed JP2: ~, wmk:1X08
- removed JP3: ~, wmk:JP1
- added JP4: ~, Connector_PinHeader_2.54mm:PinHeader_2x05_P2.54mm_Vertical, F.Cu at (136.2, 114.5)
- added R5: 10k, Resistor_SMD:R_0603_1608Metric, F.Cu at (160.6, 67.5)
- added SW1: SW_Push, Button_Switch_THT:SW_Tactile_SPST_Angled_PTS645Vx83-2LFS, F.Cu at (154.2, 58.6)
- JP1: footprint wmk:2X05 -> Connector_PinHeader_2.54mm:PinHeader_2x05_P2.54mm_Vertical
- moved R4 28.6 mm to (134.6, 69.4)
- moved CONNECT0 28.4 mm to (134.5, 57.9)
- moved C13 14.7 mm to (153.2, 92.7)
- moved IC1 13.9 mm to (152.6, 98.5)
- moved C3 13.3 mm to (151.7, 104.3)
- moved F1 12.0 mm to (148.9, 70.6), turned to 180 degrees
- moved R3 5.85 mm to (132.6, 69.4)
- moved JP1 5.30 mm to (136.2, 88.7), turned to 180 degrees
- moved X1 5.20 mm to (143.5, 62.6)
- moved POWER0 4.41 mm to (132.5, 57.9)
Connections:
- CONNECT0 pad C: Net-(U2-PA3) -> /CONNECT
- U2 pad 21: unconnected-(U2-PB10-Pad21) -> /CONNECT
- U2 pad 29: /INUSE -> /K0
- U2 pad 32: /STATUS -> /K1
- U2 pad 38: unconnected-(U2-PA15-Pad38) -> /IRQ7
Routing:
- net /K1: track 0.00 -> 42.3 mm, vias 0 -> 1
- net /K0: track 0.00 -> 39.3 mm
- net /INUSE: track 28.9 -> 0.00 mm
- net /IRQ7: track 0.00 -> 28.7 mm, vias 0 -> 2
- net /CONNECT: track 0.00 -> 28.6 mm, vias 0 -> 1
- net /STATUS: track 27.0 -> 0.00 mm
- net /CLOCK: track 43.3 -> 69.8 mm, vias 0 -> 1
- net /DATA: track 52.9 -> 74.7 mm, vias 0 -> 1
- net /RX: track 28.1 -> 43.5 mm, vias 1 -> 0
- net Net-(POWER0-PadA): track 1.74 -> 9.74 mm
- net Net-(CONNECT0-PadA): track 2.22 -> 9.57 mm
- net /TX: track 33.8 -> 40.3 mm, vias 1 -> 0
- net /USB_DP: track 19.6 -> 24.2 mm
- net VDD: track 49.0 -> 45.0 mm
- net Net-(U2-PA3): track 27.8 -> 24.4 mm
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Other:
- board size 33.3 x 100 mm -> 32.8 x 100 mm
- board text added: "RISKYREA1200"
- board text removed: "3/5/2021"
- board text removed: "Clock"
- board text removed: "Data"
- board text removed: "Inuse"
- board text removed: "ReAmiga 1200 Mouse USB"
- board text removed: "Reset"
- board text removed: "Rx"
- board text removed: "Ststus"
- board text removed: "Tx"

Commit message: PCB changes and gerbers
Parts:
- removed J2: Conn_01x02, Connector_PinHeader_2.54mm:PinHeader_1x02_P2.54mm_Vertical
- removed R1: 100k, wmk:R0603
- J1: value Conn_01x03 -> Conn_01x04; footprint Connector_PinHeader_2.54mm:PinHeader_1x03_P2.54mm_Vertical -> Connector_PinHeader_2.54mm:PinHeader_1x04_P2.54mm_Vertical
- moved J1 4.10 mm to (158.8, 95.3), turned to 0 degrees
- moved C13 1.70 mm to (151.5, 92.8)
- moved IC1 0.73 mm to (151.9, 98.6)
Connections:
- J1 pad 1: GND -> /SWDIO
- J1 pad 2: Net-(J1-Pin_2) -> /SWCLK
- J1 pad 3: VDD -> GND
- U2 pad 44: Net-(U2-BOOT0) -> GND
Routing:
- net VCC: track 9.61 -> 19.7 mm
- net /SWDIO: track 15.7 -> 22.2 mm
- net Net-(U2-BOOT0): track 6.29 -> 0.00 mm, vias 1 -> 0
- net Net-(J1-Pin_2): track 3.20 -> 0.00 mm
- net GND: track 19.6 -> 21.3 mm, vias 8 -> 9
- net /SWCLK: track 19.5 -> 20.9 mm, vias 2 -> 1
- net VDD: track 45.0 -> 45.7 mm
Other:
- outline, holes or cut-outs redrawn
- board text added: "5V"
- board text added: "Bell End Edition"
- board text added: "CLK"
- board text added: "Check PSU"
- board text added: "DATA CLOCK IRQ7 RESET K0 GND K1 RX TX"
- board text added: "DIO"
- board text added: "FPU Included."
- board text added: "MB RIGHT RB LEFT GND DOWN 5V UP LB"
- board text removed: "NRST"
- board text removed: "SWCLK"
- board text removed: "SWDIO"
- board text removed: "VCC"

Commit message: Board review
Parts:
- removed SW1: SW_Push, Button_Switch_THT:SW_Tactile_SPST_Angled_PTS645Vx83-2LFS
- added JP2: SolderJumper_2_Open, Jumper:SolderJumper-2_P1.3mm_Open_RoundedPad1.0x1.5mm, F.Cu at (134.6, 126.5)
- added JP3: SolderJumper_2_Open, Jumper:SolderJumper-2_P1.3mm_Open_RoundedPad1.0x1.5mm, F.Cu at (137.9, 126.5)
- added PROG: SW_Push, Button_Switch_THT:SW_PUSH_6mm, F.Cu at (154.2, 60.6)
- moved R5 1.25 mm to (160.5, 68.8)
Connections:
- JP4 pad 1: /TX -> Net-(JP3-B)
- JP4 pad 2: /RX -> Net-(JP2-B)
Routing:
- net Net-(JP2-B): track 0.00 -> 13.7 mm
- net Net-(JP3-B): track 0.00 -> 12.4 mm
- net /RX: track 43.5 -> 55.4 mm
- net /TX: track 40.3 -> 50.2 mm
- net VDD: track 45.7 -> 44.9 mm
- net Net-(U2-PA3): track 24.4 -> 25.0 mm
