File: board/wmk.kicad_sch (KiCad schematic)
At the start: 25 parts, among them IC1 LM1117MPX-3.3, J1 Conn_01x03, U2 STM32F103C8T6, X1 PN87520-S

Commit message: gerbers
Parts:
- removed C10, C11: 22p, wmk:C0603, symbol wmk-eagle-import:C-EUC0603
- removed PROGRAMER0: ~, wmk:JP3Q, symbol wmk-eagle-import:JP3Q
- removed Q1: ~, wmk:HC49_S, symbol wmk-eagle-import:CRYSTALHC49S
- added J2: Conn_01x02, Connector_PinHeader_2.54mm:PinHeader_1x02_P2.54mm_Vertical, symbol Connector_Generic:Conn_01x02
- U2: footprint wmk:QFP50P900X900X160-48N -> Package_QFP:LQFP-48_7x7mm_P0.5mm
Connections:
- net SWCLK: now also J2.1 (Pin_1)
- net SWDIO: now also J2.2 (Pin_2)
- no-connect marks 17 -> 20

Commit message: initial version
Parts:
- removed JP2: ~, wmk:1X08, symbol wmk-eagle-import:PINHD-1X8
- removed JP3: ~, wmk:JP1, symbol wmk-eagle-import:JP1E
- added JP4: ~, Connector_PinHeader_2.54mm:PinHeader_2x05_P2.54mm_Vertical, symbol wmk-eagle-import:PINHD-2X5
- added R5: 10k, Resistor_SMD:R_0603_1608Metric, symbol Device:R
- added SW1: SW_Push, Button_Switch_THT:SW_Tactile_SPST_Angled_PTS645Vx83-2LFS, symbol Switch:SW_Push
- JP1: footprint wmk:2X05 -> Connector_PinHeader_2.54mm:PinHeader_2x05_P2.54mm_Vertical
Connections:
- net CLOCK: now also JP4.9
- net DATA: now also JP4.10
- net GND: now also JP4.5, SW1.1
- net RESET: now also JP4.7
- net RX: now also JP4.2
- net TX: now also JP4.1
- net VDD: now also R5.1
- net at U2.13 (PA3): now also R5.2, SW1.2; no longer CONNECT0.C
- net CONNECT: now reaches U2.21 (PB10)
- net CONNECT: now also CONNECT0.C
- net IRQ7: now reaches U2.38 (PA15)
- net IRQ7: now also JP4.8
- net INUSE renamed K0
- net K0: now also JP4.6
- net STATUS renamed K1
- net K1: now also JP4.4
- no-connect marks 20 -> 18
Other:
- moved on the sheet: CONNECT0, J2, R4

Commit message: PCB changes and gerbers
Parts:
- removed J1: Conn_01x03, Connector_PinHeader_2.54mm:PinHeader_1x03_P2.54mm_Vertical, symbol Connector_Generic:Conn_01x03
- removed J2: Conn_01x02, Connector_PinHeader_2.54mm:PinHeader_1x02_P2.54mm_Vertical, symbol Connector_Generic:Conn_01x02
- removed R1: 100k, wmk:R0603, symbol wmk-eagle-import:R-EU_0922V
- added J1: Conn_01x04, Connector_PinHeader_2.54mm:PinHeader_1x04_P2.54mm_Vertical, symbol Connector_Generic:Conn_01x04
Connections:
- net GND: now also U2.44 (BOOT0), J1.3 (Pin_3)
- net SWCLK: now also J1.2 (Pin_2)
- net SWDIO: now also J1.1 (Pin_1)
- net VCC: now also J1.4 (Pin_4)

Commit message: Board review
Parts:
- added JP2, JP3: SolderJumper_2_Open, symbol Jumper:SolderJumper_2_Open
- SW1: footprint Button_Switch_THT:SW_Tactile_SPST_Angled_PTS645Vx83-2LFS -> Button_Switch_THT:SW_PUSH_6mm
Connections:
- net RX: now also JP2.1 (A); no longer JP4.2
- net TX: now also JP3.1 (A); no longer JP4.1
- new net: JP2.2 (B), JP4.2
- new net: JP3.2 (B), JP4.1

Commit message: Update footprint properties for solder jumpers in schematic
Parts:
- JP2, JP3: footprint (none) -> Jumper:SolderJumper-2_P1.3mm_Open_RoundedPad1.0x1.5mm
Changed lines of the file:
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@@
 			)
 		)
-		(property "Footprint" ""
+		(property "Footprint" "Jumper:SolderJumper-2_P1.3mm_Open_RoundedPad1.0x1.5mm"
 			(at 104.14 196.85 0)
 			(effects
@@
 			)
 		)
-		(property "Footprint" ""
+		(property "Footprint" "Jumper:SolderJumper-2_P1.3mm_Open_RoundedPad1.0x1.5mm"
 			(at 125.73 196.85 0)
 			(effects
